File: hardware/bench_test_can/kicad/l0destar.kicad_pcb (KiCad board)
At the start: 2 copper layers, 116.2 x 89 mm, 66 parts, among them CON1 MIKROBUS_HOST_CONN, J2 Conn_01x12_Socket, J3 Conn_01x03_Pin, J4 Conn_01x18_Socket, SW2 SW_SPDT

Commit message: fix date
Other:
- board text added: "l0destar tracker v1.1-CAN bench test prototype 20260613"
- board text removed: "l0destar tracker v1.1-CAN bench test prototype 20260607"
