File: hardware/prototype2.1_mini/l0destar.kicad_pcb (KiCad board)
At the start: 2 copper layers, 87.5 x 68 mm, 91 parts

Commit message: fix LED footprint and mount 5 of them vertically
Parts:
- removed S1D1, S1D2, S1D3: LED, LED_SMD:LED_0805_2012Metric
- removed S1R4, S1R5, S1R6: 1K, Resistor_SMD:R_0805_2012Metric
- added S13D1: LED, LED_SMD:LED_0603_1608Metric, F.Cu at (88.8, 110.3)
- added S13D2: LED, LED_SMD:LED_0603_1608Metric, F.Cu at (90.6, 110.3)
- added S13D3: LED, LED_SMD:LED_0603_1608Metric, F.Cu at (92.4, 110.3)
- added S13D4: LED, LED_SMD:LED_0603_1608Metric, F.Cu at (94.2, 110.3)
- added S13D5: LED, LED_SMD:LED_0603_1608Metric, F.Cu at (96.0, 110.3)
- added S13R1: 1K, Resistor_SMD:R_0805_2012Metric, F.Cu at (36.8, 103.0)
- added S13R2: 1K, Resistor_SMD:R_0805_2012Metric, F.Cu at (40.6, 103.0)
- added S13R3: 1K, Resistor_SMD:R_0805_2012Metric, F.Cu at (44.3, 103.0)
- added S13R4: 1K, Resistor_SMD:R_0805_2012Metric, F.Cu at (48.1, 103.0)
- added S13R5: 1K, Resistor_SMD:R_0805_2012Metric, F.Cu at (51.9, 103.0)
Connections:
- S1J2 pad 5: Net-(S1J2-P9) -> LED1
- S1J2 pad 6: Net-(S1J2-Pin_6) -> LED2
- S1J2 pad 7: Net-(S1J2-Pin_7) -> LED3
- S1J2 pad 8: unconnected-(S1J2-Pin_8-Pad8) -> LED4
- S1J2 pad 9: unconnected-(S1J2-Pin_9-Pad9) -> LED5
Routing:
- net Net-(S1D3-A): track 63.6 -> 0.00 mm
- net Net-(S1D2-A): track 62.3 -> 0.00 mm
- net Net-(S1D1-A): track 60.8 -> 0.00 mm
- net Net-(S13D1-A): track 0.00 -> 59.1 mm
- net Net-(S13D4-A): track 0.00 -> 58.9 mm
- net Net-(S13D2-A): track 0.00 -> 58.4 mm
- net Net-(S13D3-A): track 0.00 -> 58.0 mm
- net Net-(S13D5-A): track 0.00 -> 51.4 mm
- net LED4: track 0.00 -> 4.68 mm
- net LED5: track 0.00 -> 4.30 mm
- net LED3: track 0.00 -> 3.97 mm
- net Net-(S1J2-Pin_7): track 3.97 -> 0.00 mm
- net Net-(S1J2-Pin_6): track 3.55 -> 0.00 mm
- net LED2: track 0.00 -> 3.55 mm
- net Net-(S1J2-P9): track 3.17 -> 0.00 mm
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