File: hardware/l0destar_v2.5_micro/main_power_input.kicad_sch (KiCad schematic)
At the start: 8 parts

Commit message: fix TVS part
Parts:
- S2D2, S2D4: value PTVS30VS1UTR,115 -> PTVS33VS1UTR,115
Changed lines of the file:
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@@
 			)
 		)
-		(property "Value" "PTVS30VS1UTR,115"
+		(property "Value" "PTVS33VS1UTR,115"
 			(at 49.53 58.42 0)
 			(show_name no)
@@
 			)
 		)
-		(property "Value" "PTVS30VS1UTR,115"
+		(property "Value" "PTVS33VS1UTR,115"
 			(at 40.64 93.9799 90)
 			(show_name no)
