File: hardware/l0destar_v2.5_micro/can_interface.kicad_sch (KiCad schematic)
At the start: 14 parts

Commit message: tweaked layouts
Parts:
- S9C6: renamed from S9C5; symbol Device:C -> Device:C_Polarized
- renumbered S9C1 to S9C2, S9C4 to S9C5, S9C2 to S9C7, S9C3 to S9C8, S9U3 to S9U4
Changed lines of the file:
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@@
 		(in_pos_files yes)
 		(dnp no)
-		(property "Reference" "S9C2"
+		(property "Reference" "S9C7"
 			(at 58.674 147.574 0)
 			(show_name no)
@@
 			(project "l0destar"
 				(path "/da570340-c25f-43d9-9e24-f16e4364f6bf"
-					(reference "S9C2")
+					(reference "S9C7")
 					(unit 1)
 				)
@@
 		(dnp no)
 		(fields_autoplaced yes)
-		(property "Reference" "S9U3"
+		(property "Reference" "S9U4"
 			(at 59.69 60.96 0)
 			(show_name no)
@@
 			(project "l0destar"
 				(path "/da570340-c25f-43d9-9e24-f16e4364f6bf"
-					(reference "S9U3")
+					(reference "S9U4")
 					(unit 1)
 				)
@@
 		(in_pos_files yes)
 		(dnp no)
-		(property "Reference" "S9C3"
+		(property "Reference" "S9C8"
 			(at 70.104 147.574 0)
 			(show_name no)
@@
 			(project "l0destar"
 				(path "/da570340-c25f-43d9-9e24-f16e4364f6bf"
-					(reference "S9C3")
-					(unit 1)
-				)
-			)
-		)
-	)
-	(symbol
-		(lib_id "Device:C")
+					(reference "S9C8")
+					(unit 1)
+				)
+			)
+		)
+	)
+	(symbol
+		(lib_id "Device:C_Polarized")
 		(at 153.67 130.81 0)
 		(unit 1)
@@
 		(dnp no)
 		(fields_autoplaced yes)
-		(property "Reference" "S9C5"
-			(at 157.48 129.5399 0)
+		(property "Reference" "S9C6"
+			(at 157.48 128.6509 0)
 			(show_name no)
 			(do_not_autoplace no)
@@
 		)
 		(property "Value" "10uF"
-			(at 157.48 132.0799 0)
+			(at 157.48 131.1909 0)
 			(show_name no)
 			(do_not_autoplace no)
@@
 			)
 		)
-		(property "Description" "Unpolarized capacitor"
+		(property "Description" "Polarized capacitor"
 			(at 153.67 130.81 0)
 			(hide yes)
@@
 			(project "l0destar"
 				(path "/da570340-c25f-43d9-9e24-f16e4364f6bf"
-					(reference "S9C5")
+					(reference "S9C6")
 					(unit 1)
 				)
@@
 		(in_pos_files yes)
 		(dnp no)
-		(property "Reference" "S9C4"
+		(property "Reference" "S9C5"
 			(at 143.764 129.794 0)
 			(show_name no)
@@
 			(project "l0destar"
 				(path "/da570340-c25f-43d9-9e24-f16e4364f6bf"
-					(reference "S9C4")
+					(reference "S9C5")
 					(unit 1)
 				)
@@
 		(in_pos_files yes)
 		(dnp no)
-		(property "Reference" "S9C1"
+		(property "Reference" "S9C2"
 			(at 119.38 28.448 0)
 			(show_name no)
@@
 			(project "l0destar"
 				(path "/da570340-c25f-43d9-9e24-f16e4364f6bf"
-					(reference "S9C1")
-					(unit 1)
-				)
+					(reference "S9C2")
+					(unit 1)
+				)
