File: hardware/l0destar_v2.5_micro/l0destar.kicad_sch (KiCad schematic)
At the start: 10 parts

Commit message: fix references
Parts:
- renumbered C2 to S1C1, C3 to S1C2
Changed lines of the file:
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@@
 		(dnp no)
 		(fields_autoplaced yes)
-		(property "Reference" "C3"
+		(property "Reference" "S1C2"
 			(at 63.5 80.0099 0)
 			(show_name no)
@@
 			(project "l0destar"
 				(path "/463fa308-d92b-480b-9c45-50693d427ea2"
-					(reference "C3")
+					(reference "S1C2")
 					(unit 1)
 				)
@@
 		(dnp no)
 		(fields_autoplaced yes)
-		(property "Reference" "C2"
+		(property "Reference" "S1C1"
 			(at 48.26 80.0099 0)
 			(show_name no)
@@
 			(project "l0destar"
 				(path "/463fa308-d92b-480b-9c45-50693d427ea2"
-					(reference "C2")
+					(reference "S1C1")
 					(unit 1)
 				)

Commit message: tweaked layouts
Parts:
- removed S1NT1: NetTie_2, symbol Device:NetTie_2
- removed S1R3: 100K, Resistor_SMD:R_0402_1005Metric, symbol Device:R
Connections:
- net VSYS: no longer names the net of S1J2.2 (VSYS)
