File: hardware/l0destar_v3.0/iso-9141_interface.kicad_sch (KiCad schematic)
At the start: 12 parts

Commit message: updated v3.0 part specifications and added to the schematics
Parts:
- S10C1: value 100nF -> 0402 100nF 50V 10% X7R
- S10R1, S10R2, S10R5: value 10K -> 0402 10K 1%
- S10R3, S10R4: value 510R -> 2512 510R 1% 2W
Other:
- moved on the sheet: S10C1, S10D1, S10Q1, S10R3

Commit message: fix discrepencies
Parts:
- S10R1, S10R2, S10R5: value 0402 10K 1% -> 0402 10K 5%
- S10R3, S10R4: value 2512 510R 1% 2W -> 2512 510R 5% 2W
Changed lines of the file:
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@@
 			)
 		)
-		(property "Value" "0402 10K 1%"
+		(property "Value" "0402 10K 5%"
 			(at 61.976 35.56 90)
 			(show_name no)
@@
 			)
 		)
-		(property "Value" "2512 510R 1% 2W"
+		(property "Value" "2512 510R 5% 2W"
 			(at 116.84 51.435 0)
 			(show_name no)
@@
 			)
 		)
-		(property "Value" "0402 10K 1%"
+		(property "Value" "0402 10K 5%"
 			(at 49.276 66.04 90)
 			(show_name no)
@@
 			)
 		)
-		(property "Value" "2512 510R 1% 2W"
+		(property "Value" "2512 510R 5% 2W"
 			(at 37.465 102.87 0)
 			(show_name no)
@@
 			)
 		)
-		(property "Value" "0402 10K 1%"
+		(property "Value" "0402 10K 5%"
 			(at 77.47 123.1899 0)
 			(show_name no)
