File: hardware/l0destar_v3.0/main_power_input.kicad_sch (KiCad schematic)
At the start: 9 parts

Commit message: updated v3.0 part specifications and added to the schematics
Parts:
- S2C1: value CKG57NX7R1H476M500JH - 47uF -> 47uF 2220 50V 20% X7R
- S2Q1, S2Q2: value SQ2361 -> SQ2361ES-T1_GE3
- S2R1: value 1M -> 0402 1M 1%
- S2R2: value 10M -> 0402 10M 1%
Changed lines of the file:
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@@
 			)
 		)
-		(property "Value" "CKG57NX7R1H476M500JH - 47uF"
+		(property "Value" "47uF 2220 50V 20% X7R"
 			(at 106.68 93.9799 90)
 			(show_name no)
@@
 			)
 		)
-		(property "Datasheet" ""
+		(property "Datasheet" "CKG57NX7R1H476M500JH"
 			(at 102.87 91.44 0)
 			(hide yes)
@@
 			)
 		)
-		(property "Value" "SQ2361"
+		(property "Value" "SQ2361ES-T1_GE3"
 			(at 63.5 36.83 90)
 			(show_name no)
@@
 			)
 		)
-		(property "Value" "1M"
+		(property "Value" "0402 1M 1%"
 			(at 66.04 58.4199 0)
 			(show_name no)
@@
 			)
 		)
-		(property "Value" "10M"
+		(property "Value" "0402 10M 1%"
 			(at 66.04 100.3299 0)
 			(show_name no)
@@
 			)
 		)
-		(property "Value" "SQ2361"
+		(property "Value" "SQ2361ES-T1_GE3"
 			(at 63.5 80.01 90)
 			(show_name no)

Commit message: fix discrepencies
Parts:
- S2R1: value 0402 1M 1% -> 0402 1M 5%
- S2R2: value 0402 10M 1% -> 0402 10M 5%
Changed lines of the file:
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@@
 			)
 		)
-		(property "Value" "0402 1M 1%"
+		(property "Value" "0402 1M 5%"
 			(at 66.04 58.4199 0)
 			(show_name no)
@@
 			)
 		)
-		(property "Value" "0402 10M 1%"
+		(property "Value" "0402 10M 5%"
 			(at 66.04 100.3299 0)
 			(show_name no)

Commit message: fix pulldown resistor spec
Parts:
- S2R2: value 0402 10M 5% -> 0402 1M 5%
Changed lines of the file:
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@@
 			)
 		)
-		(property "Value" "0402 10M 5%"
+		(property "Value" "0402 1M 5%"
 			(at 66.04 100.3299 0)
 			(show_name no)
