File: hardware/l0destar_v2.5_can/auxillary_power_control.kicad_sch (KiCad schematic)
At the start: 6 parts

Commit message: tweaked layouts
Parts:
- renumbered S7Q3 to S7Q1, S7Q4 to S7Q2, S7R5 to S7R1, S7R6 to S7R2, S7R7 to S7R3, S7R8 to S7R4
Changed lines of the file:
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@@
 		(dnp no)
 		(fields_autoplaced yes)
-		(property "Reference" "S7Q4"
+		(property "Reference" "S7Q2"
 			(at 120.65 30.48 90)
 			(show_name no)
@@
 			(project "l0destar"
 				(path "/6b82df34-c34f-4615-8477-25790583a5d0"
-					(reference "S7Q4")
+					(reference "S7Q2")
 					(unit 1)
 				)
@@
 		(in_pos_files yes)
 		(dnp no)
-		(property "Reference" "S7Q3"
+		(property "Reference" "S7Q1"
 			(at 84.328 34.798 0)
 			(show_name no)
@@
 			(project "l0destar"
 				(path "/6b82df34-c34f-4615-8477-25790583a5d0"
-					(reference "S7Q3")
+					(reference "S7Q1")
 					(unit 1)
 				)
@@
 		(dnp no)
 		(fields_autoplaced yes)
-		(property "Reference" "S7R8"
+		(property "Reference" "S7R4"
 			(at 99.06 53.34 90)
 			(show_name no)
@@
 			(project "l0destar"
 				(path "/6b82df34-c34f-4615-8477-25790583a5d0"
-					(reference "S7R8")
+					(reference "S7R4")
 					(unit 1)
 				)
@@
 		(dnp no)
 		(fields_autoplaced yes)
-		(property "Reference" "S7R6"
+		(property "Reference" "S7R2"
 			(at 67.31 43.1799 0)
 			(show_name no)
@@
 			(project "l0destar"
 				(path "/6b82df34-c34f-4615-8477-25790583a5d0"
-					(reference "S7R6")
+					(reference "S7R2")
 					(unit 1)
 				)
@@
 		(dnp no)
 		(fields_autoplaced yes)
-		(property "Reference" "S7R5"
+		(property "Reference" "S7R1"
 			(at 57.15 31.75 90)
 			(show_name no)
@@
 			(project "l0destar"
 				(path "/6b82df34-c34f-4615-8477-25790583a5d0"
-					(reference "S7R5")
+					(reference "S7R1")
 					(unit 1)
 				)
@@
 		(dnp no)
 		(fields_autoplaced yes)
-		(property "Reference" "S7R7"
+		(property "Reference" "S7R3"
 			(at 99.06 25.4 90)
 			(show_name no)
@@
 			(project "l0destar"
 				(path "/6b82df34-c34f-4615-8477-25790583a5d0"
-					(reference "S7R7")
-					(unit 1)
-				)
+					(reference "S7R3")
+					(unit 1)
+				)
