File: hardware/l0destar_v2.5_can/buck_converter.kicad_sch (KiCad schematic)
At the start: 11 parts

Commit message: tweaked layouts
Parts:
- renumbered S6C6 to S6C1, S6C7 to S6C2, S6C8 to S6C3, S6C9 to S6C4, S6C10 to S6C5, S6L2 to S6L1, S6R4 to S6R1, S6R5 to S6R2, S6R6 to S6R3, S6U2 to S6U1, S6U3 to S6U2
Changed lines of the file:
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@@
 		(dnp no)
 		(fields_autoplaced yes)
-		(property "Reference" "S6L2"
+		(property "Reference" "S6L1"
 			(at 123.19 21.59 0)
 			(show_name no)
@@
 			(project "l0destar"
 				(path "/3b34a799-c26a-4c86-88e6-720fda4c7fd2"
-					(reference "S6L2")
+					(reference "S6L1")
 					(unit 1)
 				)
@@
 		(in_pos_files yes)
 		(dnp no)
-		(property "Reference" "S6C8"
+		(property "Reference" "S6C3"
 			(at 152.4 53.34 0)
 			(show_name no)
@@
 			(project "l0destar"
 				(path "/3b34a799-c26a-4c86-88e6-720fda4c7fd2"
-					(reference "S6C8")
+					(reference "S6C3")
 					(unit 1)
 				)
@@
 		(in_pos_files yes)
 		(dnp no)
-		(property "Reference" "S6C6"
+		(property "Reference" "S6C1"
 			(at 28.956 43.434 0)
 			(show_name no)
@@
 			(project "l0destar"
 				(path "/3b34a799-c26a-4c86-88e6-720fda4c7fd2"
-					(reference "S6C6")
+					(reference "S6C1")
 					(unit 1)
 				)
@@
 		(in_pos_files yes)
 		(dnp no)
-		(property "Reference" "S6R5"
+		(property "Reference" "S6R2"
 			(at 118.364 77.216 0)
 			(show_name no)
@@
 			(project "l0destar"
 				(path "/3b34a799-c26a-4c86-88e6-720fda4c7fd2"
-					(reference "S6R5")
+					(reference "S6R2")
 					(unit 1)
 				)
@@
 		(in_pos_files yes)
 		(dnp no)
-		(property "Reference" "S6C10"
+		(property "Reference" "S6C5"
 			(at 161.036 90.17 0)
 			(show_name no)
@@
 			(project "l0destar"
 				(path "/3b34a799-c26a-4c86-88e6-720fda4c7fd2"
-					(reference "S6C10")
+					(reference "S6C5")
 					(unit 1)
 				)
@@
 		(dnp no)
 		(fields_autoplaced yes)
-		(property "Reference" "S6U2"
+		(property "Reference" "S6U1"
 			(at 88.9 33.02 0)
 			(show_name no)
@@
 			(project "l0destar"
 				(path "/3b34a799-c26a-4c86-88e6-720fda4c7fd2"
-					(reference "S6U2")
+					(reference "S6U1")
 					(unit 1)
 				)
@@
 		(dnp no)
 		(fields_autoplaced yes)
-		(property "Reference" "S6U3"
+		(property "Reference" "S6U2"
 			(at 180.34 30.48 0)
 			(show_name no)
@@
 			(project "l0destar"
 				(path "/3b34a799-c26a-4c86-88e6-720fda4c7fd2"
-					(reference "S6U3")
+					(reference "S6U2")
 					(unit 1)
 				)
@@
 		(in_pos_files yes)
 		(dnp no)
-		(property "Reference" "S6R6"
+		(property "Reference" "S6R3"
 			(at 144.526 83.566 90)
 			(show_name no)
@@
 			(project "l0destar"
 				(path "/3b34a799-c26a-4c86-88e6-720fda4c7fd2"
-					(reference "S6R6")
+					(reference "S6R3")
 					(unit 1)
 				)
@@
 		(in_pos_files yes)
 		(dnp no)
-		(property "Reference" "S6C7"
+		(property "Reference" "S6C2"
 			(at 41.148 67.564 0)
 			(show_name no)
@@
 			(project "l0destar"
 				(path "/3b34a799-c26a-4c86-88e6-720fda4c7fd2"
-					(reference "S6C7")
+					(reference "S6C2")
 					(unit 1)
 				)
@@
 		(in_pos_files yes)
 		(dnp no)
-		(property "Reference" "S6C9"
+		(property "Reference" "S6C4"
 			(at 142.748 72.39 90)
 			(show_name no)
@@
 			(project "l0destar"
 				(path "/3b34a799-c26a-4c86-88e6-720fda4c7fd2"
-					(reference "S6C9")
+					(reference "S6C4")
 					(unit 1)
 				)
@@
 		(dnp no)
 		(fields_autoplaced yes)
-		(property "Reference" "S6R4"
+		(property "Reference" "S6R1"
 			(at 52.07 67.3099 0)
 			(show_name no)
@@
 			(project "l0destar"
 				(path "/3b34a799-c26a-4c86-88e6-720fda4c7fd2"
-					(reference "S6R4")
-					(unit 1)
-				)
+					(reference "S6R1")
+					(unit 1)
+				)
