File: hardware/l0destar_v2.5_kline/l0destar.kicad_sch (KiCad schematic)
At the start: 10 parts

Commit message: tweaked layouts
Parts:
- removed S1NT1: NetTie_2, symbol Device:NetTie_2
- removed S1R3: 100K, Resistor_SMD:R_0402_1005Metric, symbol Device:R
Connections:
- net VSYS: no longer names the net of S1J2.2 (VSYS)
