File: hardware/l0destar_v2.5_kline/l0destar.kicad_pcb (KiCad board)
At the start: 4 copper layers, 66.7 x 37.5 mm, 112 parts

Commit message: tweaked layouts
Parts:
- removed S1R3: 100K, Resistor_SMD:R_0402_1005Metric
- S10D1, S10D2, S2D2, S2D4: value PTVS30VS1UTR,115 -> PTVS33VS1UTR,115
- renumbered S10C4 to S10C1, S10C1 to S10C2, S10C2 to S10C4, S10R10 to S10R1, S10R7 to S10R2, S10R9 to S10R3, C2 to S1C1, C3 to S1C2, S6C6 to S6C1, S6C15 to S6C10, S6C7 to S6C2, S6C8 to S6C3, S6C9 to S6C4, S6C10 to S6C5, S6C11 to S6C6, S6C12 to S6C7, S6C14 to S6C8, S6C13 to S6C9, S6L2 to S6L1, S6L3 to S6L2, S6R4 to S6R1, S6R5 to S6R2, S6R6 to S6R3, S6R7 to S6R4, S6R8 to S6R5, S6R9 to S6R6, S6U2 to S6U1, S6U3 to S6U2, S6U4 to S6U3, S6U5 to S6U4, S7Q3 to S7Q1, S7Q4 to S7Q2, S7Q5 to S7Q3, S7Q6 to S7Q4, S7R5 to S7R1, S7R6 to S7R2, S7R7 to S7R3, S7R8 to S7R4, S7R9 to S7R5, S7R10 to S7R6, S7R11 to S7R7, S7R12 to S7R8
Connections:
- S1J2 pad 2: VSYS -> unconnected-(S1J2-VSYS-Pad2)
- S1J2 pad 4: Net-(S1J2-ENABLE) -> unconnected-(S1J2-ENABLE-Pad4)
Routing:
- net GND: track 98.3 -> 94.7 mm, vias 206 -> 173
- net VSYS: track 3.45 -> 0.00 mm
- net Net-(S1J2-ENABLE): track 3.13 -> 0.00 mm
Other:
- board text removed: "ENABLE"
- board text removed: "VSYS"

Commit message: update testing
Parts:
- added S10R4: 510R, Resistor_SMD:R_2512_6332Metric, F.Cu at (70.4, 77.7)
- moved S10R2 0.53 mm to (66.3, 77.7)
Routing:
- net ISO9141_L: track 71.5 -> 82.9 mm, vias 3 -> 5
- net PP12VK: track 42.9 -> 45.3 mm

Commit message: fix bias tee cap ordering on all boards
Parts:
- moved S15C4 2.18 mm to (78.8, 84.9)
- moved S15C2 1.09 mm to (81.0, 84.9)
- moved S15C3 1.09 mm to (79.9, 84.9)
