File: hardware/l0destar_v3.1/accelerometer.kicad_sch (KiCad schematic)
At the start: 4 parts

Commit message: update v3.1
Parts:
- S8C2: value 0603 10uF 10V 20% X7T -> 0603 10uF 10V 20% X7R
Changed lines of the file:
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@@
 			)
 		)
-		(property "Value" "0603 10uF 10V 20% X7T"
+		(property "Value" "0603 10uF 10V 20% X7R"
 			(at 152.146 48.26 0)
 			(show_name no)

Commit message: update v3.1
Parts:
- S8C1, S8C3: Manufacturer_Name (none) -> Multicomp Pro; Manufacturer_Part_Number (none) -> MC0402B104K250CT
- S8C2: Manufacturer_Name (none) -> TDK; Manufacturer_Part_Number (none) -> C1608X7R1A106M080AT
- S8U1: Availability In Stock -> (none); Check_prices https://www.snapeda.com/parts/ASM330LHHXTR/STMicroelectroni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 -> (none); MF STMicroelectronics -> (none); MP ASM330LHHXTR -> (none); Manufacturer_Name (none) -> STMicroelectronics; Manufacturer_Part_Number (none) -> ASM330LHHXTR; Package VFLGA-14 STMicroelectronics -> (none); Price None -> (none); SnapEDA_Link https://www.snapeda.com/parts/ASM330LHHXTR/STMicroelectroni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 -> (none)
Changed lines of the file:
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@@
 			)
 		)
-		(property "Datasheet" ""
+		(property "Datasheet" "https://product.tdk.com/en/search/capacitor/ceramic/mlcc/info?part_no=C1608X7R1A106M080AT"
 			(at 151.13 41.91 0)
 			(hide yes)
@@
 					(size 1.27 1.27)
 				)
+			)
+		)
+		(property "Manufacturer_Part_Number" "C1608X7R1A106M080AT"
+			(at 151.13 41.91 0)
+			(hide yes)
+			(show_name no)
+			(do_not_autoplace no)
+			(effects
+				(font
+					(size 1.27 1.27)
+				)
+				(justify left top)
+			)
+		)
+		(property "Manufacturer_Name" "TDK"
+			(at 151.13 41.91 0)
+			(hide yes)
+			(show_name no)
+			(do_not_autoplace no)
+			(effects
+				(font
+					(size 1.27 1.27)
+				)
+				(justify left top)
 			)
 		)
@@
 			)
 		)
-		(property "Datasheet" ""
+		(property "Datasheet" "https://uk.farnell.com/multicomp-pro/mc0402b104k250ct/cap-0-1-f-25v-10-x7r-0402/dp/2320759"
 			(at 121.92 41.91 0)
 			(hide yes)
@@
 					(size 1.27 1.27)
 				)
+			)
+		)
+		(property "Manufacturer_Part_Number" "MC0402B104K250CT"
+			(at 121.92 41.91 0)
+			(hide yes)
+			(show_name no)
+			(do_not_autoplace no)
+			(effects
+				(font
+					(size 1.27 1.27)
+				)
+				(justify left top)
+			)
+		)
+		(property "Manufacturer_Name" "Multicomp Pro"
+			(at 121.92 41.91 0)
+			(hide yes)
+			(show_name no)
+			(do_not_autoplace no)
+			(effects
+				(font
+					(size 1.27 1.27)
+				)
+				(justify left top)
 			)
 		)
@@
 			)
 		)
-		(property "Datasheet" ""
+		(property "Datasheet" "https://uk.farnell.com/multicomp-pro/mc0402b104k250ct/cap-0-1-f-25v-10-x7r-0402/dp/2320759"
 			(at 87.63 40.64 0)
 			(hide yes)
@@
 					(size 1.27 1.27)
 				)
+			)
+		)
+		(property "Manufacturer_Part_Number" "MC0402B104K250CT"
+			(at 87.63 40.64 0)
+			(hide yes)
+			(show_name no)
+			(do_not_autoplace no)
+			(effects
+				(font
+					(size 1.27 1.27)
+				)
+				(justify left top)
+			)
+		)
+		(property "Manufacturer_Name" "Multicomp Pro"
+			(at 87.63 40.64 0)
+			(hide yes)
+			(show_name no)
+			(do_not_autoplace no)
+			(effects
+				(font
+					(size 1.27 1.27)
+				)
+				(justify left top)
 			)
 		)
@@
 			)
 		)
-		(property "Datasheet" ""
+		(property "Datasheet" "https://www.st.com/resource/en/datasheet/asm330lhhx.pdf"
 			(at 58.42 46.99 0)
 			(hide yes)
@@
 			)
 		)
-		(property "MF" "STMicroelectronics"
+		(property "Manufacturer_Name" "STMicroelectronics"
 			(at 58.42 46.99 0)
 			(hide yes)
@@
 			)
 		)
-		(property "Package" "VFLGA-14 STMicroelectronics"
-			(at 58.42 46.99 0)
-			(hide yes)
-			(show_name no)
-			(do_not_autoplace no)
-			(effects
-				(font
-					(size 1.27 1.27)
-				)
-				(justify bottom)
-			)
-		)
-		(property "Price" "None"
-			(at 58.42 46.99 0)
-			(hide yes)
-			(show_name no)
-			(do_not_autoplace no)
-			(effects
-				(font
-					(size 1.27 1.27)
-				)
-				(justify bottom)
-			)
-		)
-		(property "Check_prices" "https://www.snapeda.com/parts/ASM330LHHXTR/STMicroelectronics/view-part/?ref=eda"
-			(at 58.42 46.99 0)
-			(hide yes)
-			(show_name no)
-			(do_not_autoplace no)
-			(effects
-				(font
-					(size 1.27 1.27)
-				)
-				(justify bottom)
-			)
-		)
 		(property "STANDARD" "Manufacturer Recommendations"
 			(at 58.42 46.99 0)
@@
 			)
 		)
-		(property "SnapEDA_Link" "https://www.snapeda.com/parts/ASM330LHHXTR/STMicroelectronics/view-part/?ref=snap"
-			(at 58.42 46.99 0)
-			(hide yes)
-			(show_name no)
-			(do_not_autoplace no)
-			(effects
-				(font
-					(size 1.27 1.27)
-				)
-				(justify bottom)
-			)
-		)
-		(property "MP" "ASM330LHHXTR"
-			(at 58.42 46.99 0)
-			(hide yes)
-			(show_name no)
-			(do_not_autoplace no)
-			(effects
-				(font
-					(size 1.27 1.27)
-				)
-				(justify bottom)
-			)
-		)
-		(property "Availability" "In Stock"
-			(at 58.42 46.99 0)
-			(hide yes)
+		(property "Manufacturer_Part_Number" "ASM330LHHXTR"
+			(at 58.42 46.99 0)
+			(hide yes)

Commit message: update sheet annotations
Other:
- note added: "19/08/2026"
- note added: "3.1"
- note added: "ASM330LHHXTR 6-axis IMU 100pF decoupling caps on SDA/SCL (paired with 1.8K pullups on the connector sheet) Optional ferrite bead filter (0R 0402 by default)"
- note removed: "1.0"
- note removed: "30/05/2026"
- note removed: "ASM330LHHXG1TR 6-axis IMU 3-axis accelerometer 3-axis gyroscope Connects to the I2C bus"
Changed lines of the file:
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@@
 	(generator_version "10.0")
 	(paper "A4")
-	(text "30/05/2026"
+	(text "19/08/2026"
 		(exclude_from_sim no)
 		(at 206.248 193.294 0)
@@
 		)
 	)
-	(text "ASM330LHHXG1TR 6-axis IMU\n3-axis accelerometer\n3-axis gyroscope\nConnects to the I2C bus"
+	(text "ASM330LHHXTR 6-axis IMU\n100pF decoupling caps on SDA/SCL (paired with 1.8K pullups on the connector sheet)\nOptional ferrite bead filter (0R 0402 by default)"
 		(exclude_from_sim no)
-		(at 180.34 172.974 0)
+		(at 179.07 170.815 0)
 		(effects
 			(font
@@
 		)
 	)
-	(text "1.0"
+	(text "3.1"
 		(exclude_from_sim no)
 		(at 268.224 193.294 0)

Commit message: schematic<>readme discrepency fixes
Parts:
- S8C1, S8C3: value 0402 100nF 10V 10% X7R -> 0402 100nF 50V 10% X7R; Manufacturer_Name Multicomp Pro -> Murata; Manufacturer_Part_Number MC0402B104K250CT -> GRM155R71H104KE14D
Other:
- note added: "ASM330LHHXTR 6-axis IMU 100nF decoupling caps on SDA/SCL (paired with 1.8K pullups on the connector sheet) Optional ferrite bead filter (0R 0402 by default)"
- note removed: "ASM330LHHXTR 6-axis IMU 100pF decoupling caps on SDA/SCL (paired with 1.8K pullups on the connector sheet) Optional ferrite bead filter (0R 0402 by default)"
Changed lines of the file:
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@@
 		)
 	)
-	(text "ASM330LHHXTR 6-axis IMU\n100pF decoupling caps on SDA/SCL (paired with 1.8K pullups on the connector sheet)\nOptional ferrite bead filter (0R 0402 by default)"
+	(text "ASM330LHHXTR 6-axis IMU\n100nF decoupling caps on SDA/SCL (paired with 1.8K pullups on the connector sheet)\nOptional ferrite bead filter (0R 0402 by default)"
 		(exclude_from_sim no)
 		(at 179.07 170.815 0)
@@
 			)
 		)
-		(property "Value" "0402 100nF 10V 10% X7R"
+		(property "Value" "0402 100nF 50V 10% X7R"
 			(at 122.936 48.26 0)
 			(show_name no)
@@
 			)
 		)
-		(property "Datasheet" "https://uk.farnell.com/multicomp-pro/mc0402b104k250ct/cap-0-1-f-25v-10-x7r-0402/dp/2320759"
+		(property "Datasheet" ""
 			(at 121.92 41.91 0)
 			(hide yes)
@@
 			)
 		)
-		(property "Description" "Unpolarized capacitor"
+		(property "Description" ""
 			(at 121.92 41.91 0)
 			(hide yes)
@@
 			)
 		)
-		(property "Manufacturer_Part_Number" "MC0402B104K250CT"
+		(property "Manufacturer_Part_Number" "GRM155R71H104KE14D"
 			(at 121.92 41.91 0)
 			(hide yes)
@@
 			)
 		)
-		(property "Manufacturer_Name" "Multicomp Pro"
+		(property "Manufacturer_Name" "Murata"
 			(at 121.92 41.91 0)
 			(hide yes)
@@
 			)
 		)
-		(property "Value" "0402 100nF 10V 10% X7R"
+		(property "Value" "0402 100nF 50V 10% X7R"
 			(at 91.44 42.164 0)
 			(show_name no)
@@
 			)
 		)
-		(property "Datasheet" "https://uk.farnell.com/multicomp-pro/mc0402b104k250ct/cap-0-1-f-25v-10-x7r-0402/dp/2320759"
+		(property "Datasheet" ""
 			(at 87.63 40.64 0)
 			(hide yes)
@@
 			)
 		)
-		(property "Description" "Unpolarized capacitor"
+		(property "Description" ""
 			(at 87.63 40.64 0)
 			(hide yes)
@@
 			)
 		)
-		(property "Manufacturer_Part_Number" "MC0402B104K250CT"
+		(property "Manufacturer_Part_Number" "GRM155R71H104KE14D"
 			(at 87.63 40.64 0)
 			(hide yes)
@@
 			)
 		)
-		(property "Manufacturer_Name" "Multicomp Pro"
+		(property "Manufacturer_Name" "Murata"
 			(at 87.63 40.64 0)
 			(hide yes)
