File: hardware/l0destar_v3.1/buck_converter.kicad_sch (KiCad schematic)
At the start: 14 parts

Commit message: update v3.1
Parts:
- S6C4: value 0402 10pF 10V X7R -> 0402 10pF 10V C0G/NP0
- S6C5: value 0805 22uF 10V 20% X7T -> 0805 22uF 10V 20% X7R
Changed lines of the file:
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@@
 			)
 		)
-		(property "Value" "0805 22uF 10V 20% X7T"
+		(property "Value" "0805 22uF 10V 20% X7R"
 			(at 158.496 99.06 0)
 			(show_name no)
@@
 			)
 		)
-		(property "Value" "0402 10pF 10V X7R"
+		(property "Value" "0402 10pF 10V C0G/NP0"
 			(at 141.478 82.55 90)
 			(show_name no)

Commit message: update v3.1
Parts:
- S6C1: Manufacturer_Name (none) -> Multicomp Pro; Manufacturer_Part_Number (none) -> MC0402B104K250CT
- S6C2: Manufacturer_Name (none) -> Kyocera AVX; Manufacturer_Part_Number (none) -> KAM05CR71A105KH
- S6C3: Manufacturer_Name (none) -> Murata; Manufacturer_Part_Number (none) -> GRM21BZ71H475KE15K
- S6C4: Manufacturer_Name (none) -> Kemet; Manufacturer_Part_Number (none) -> C0402C100K5RACTU
- S6C5: Manufacturer_Name (none) -> Cal-Chip Electronics; Manufacturer_Part_Number (none) -> GMC21X7R226M10NT
- S6C6, S6C7: Manufacturer_Name (none) -> Samsung Electro-Mechanics; Manufacturer_Part_Number (none) -> CL32B476MPJNNNE
- S6C8: Manufacturer_Name (none) -> Taiyo Yuden; Manufacturer_Part_Number (none) -> MCASU105SB7104KFNA01
- S6L1: Availability In Stock -> (none); Check_prices https://www.snapeda.com/parts/XFL4020-222ME/Coilcraft/view-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 -> (none); MF Coilcraft -> (none); MP XFL4020-222ME -> (none); Manufacturer_Name (none) -> Coilcraft; Manufacturer_Part_Number (none) -> XFL4020-222MEC; Package None -> (none); Price None -> (none); SnapEDA_Link https://www.snapeda.com/parts/XFL4020-222ME/Coilcraft/view-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 -> (none)
- S6R1: Manufacturer_Name (none) -> Yageo; Manufacturer_Part_Number (none) -> RC0402FR-0718K2L
- S6R2: Manufacturer_Name (none) -> Multicomp Pro; Manufacturer_Part_Number (none) -> MCMR04X2263FTL
- S6R3: Manufacturer_Name (none) -> Panasonic; Manufacturer_Part_Number (none) -> ERJ2RKF1004X
- S6U1: Availability In Stock -> (none); Check_prices https://www.snapeda.com/parts/LT8609AIMSE%23PBF/Analog+Devi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 -> (none); MANUFACTURER_PART_NUMBER lt8609hmse#trpbf -> (none); MF Analog Devices -> (none); MP LT8609AIMSE#PBF -> (none); Manufacturer_Name (none) -> Analog Devices; Manufacturer_Part_Number (none) -> LT8609AIMSE#PBF; Package MSOP-10 Linear Technology -> (none); Price None -> (none); SnapEDA_Link https://www.snapeda.com/parts/LT8609AIMSE%23PBF/Analog+Devi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 -> (none)
- S6U2: Manufacturer_Name (none) -> Texas Instruments; Manufacturer_Part_Number (none) -> LM66100

Commit message: update sheet annotations
Other:
- note added: "19/08/2026"
- note added: "3.1"
- note added: "Buck converter 12V -> 4.2V LT8609 reference implementation LM66100 ideal diode on the output side to prevent USB voltage flowing backwards Bulk ceramics on the output"
- note removed: "1.0"
- note removed: "30/05/2026"
- note removed: "Buck converter 12V -> 4.2V LT8609 reference implementation LM66100 ideal diode on the output side to prevent USB voltage flowing backwards"
Changed lines of the file:
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@@
 	(generator_version "10.0")
 	(paper "A4")
-	(text "30/05/2026"
+	(text "19/08/2026"
 		(exclude_from_sim no)
 		(at 205.994 193.294 0)
@@
 		)
 	)
-	(text "Buck converter 12V -> 4.2V\nLT8609 reference implementation\nLM66100 ideal diode on the output side to prevent USB voltage flowing backwards"
+	(text "Buck converter 12V -> 4.2V\nLT8609 reference implementation\nLM66100 ideal diode on the output side to prevent USB voltage flowing backwards\nBulk ceramics on the output"
 		(exclude_from_sim no)
 		(at 180.848 172.466 0)
@@
 		)
 	)
-	(text "1.0"
+	(text "3.1"
 		(exclude_from_sim no)
 		(at 268.478 193.294 0)

Commit message: schematic<>readme discrepency fixes
Parts:
- S6C1: value 0402 100nF 25V 10% X7R -> 0402 100nF 50V 10% X7R; Manufacturer_Name Multicomp Pro -> Murata; Manufacturer_Part_Number MC0402B104K250CT -> GRM155R71H104KE14D
- S6C4: value 0402 10pF 10V C0G/NP0 -> 0402 10pF 50V C0G/NP0
- S6C8: Manufacturer_Name Taiyo Yuden -> Murata; Manufacturer_Part_Number MCASU105SB7104KFNA01 -> GRM155R71H104KE14D
Changed lines of the file:
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@@
 			)
 		)
-		(property "Value" "0402 100nF 25V 10% X7R"
+		(property "Value" "0402 100nF 50V 10% X7R"
 			(at 28.956 43.434 0)
 			(show_name no)
@@
 			)
 		)
-		(property "Datasheet" "https://uk.farnell.com/multicomp-pro/mc0402b104k250ct/cap-0-1-f-25v-10-x7r-0402/dp/2320759"
+		(property "Datasheet" ""
 			(at 25.4 41.91 0)
 			(hide yes)
@@
 			)
 		)
-		(property "Description" "Unpolarized capacitor"
+		(property "Description" ""
 			(at 25.4 41.91 0)
 			(hide yes)
@@
 			)
 		)
-		(property "Manufacturer_Part_Number" "MC0402B104K250CT"
+		(property "Manufacturer_Part_Number" "GRM155R71H104KE14D"
 			(at 25.4 41.91 0)
 			(hide yes)
@@
 			)
 		)
-		(property "Manufacturer_Name" "Multicomp Pro"
+		(property "Manufacturer_Name" "Murata"
 			(at 25.4 41.91 0)
 			(hide yes)
@@
 			)
 		)
-		(property "Datasheet" "https://ds.yuden.co.jp/TYCOMPAS/or/detail?pn=MCASU105SB7104KFNA01&u=M"
+		(property "Datasheet" ""
 			(at 167.64 63.5 0)
 			(hide yes)
@@
 			)
 		)
-		(property "Description" "Unpolarized capacitor"
+		(property "Description" ""
 			(at 167.64 63.5 0)
 			(hide yes)
@@
 			)
 		)
-		(property "Manufacturer_Part_Number" "MCASU105SB7104KFNA01"
+		(property "Manufacturer_Part_Number" "GRM155R71H104KE14D"
 			(at 167.64 63.5 0)
 			(hide yes)
@@
 			)
 		)
-		(property "Manufacturer_Name" "Taiyo Yuden"
+		(property "Manufacturer_Name" "Murata"
 			(at 167.64 63.5 0)
 			(hide yes)
@@
 			)
 		)
-		(property "Value" "0402 10pF 10V C0G/NP0"
+		(property "Value" "0402 10pF 50V C0G/NP0"
 			(at 141.478 82.55 90)
 			(show_name no)
