File: hardware/l0destar_v3.1/l0destar.kicad_sch (KiCad schematic)
At the start: 8 parts

Commit message: minor tweaks
Parts:
- added S1C1: 0402 100nF 10V 10% X7R, Capacitor_SMD:C_0402_1005Metric, symbol Device:C
Connections:
- net GND: now also S1C1.1
- net PP4V2: now also S1C1.2
Changed lines of the file:
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@@
 		(color 0 0 0 0)
 	)
+	(junction
+		(at 45.085 68.58)
+		(diameter 0)
+		(color 0 0 0 0)
+	)
 	(wire
 		(pts
@@
 	(wire
 		(pts
+			(xy 45.085 78.105) (xy 45.085 81.28)
+		)
+		(stroke
+			(width 0)
+			(type default)
+		)
+	)
+	(wire
+		(pts
 			(xy 124.46 88.9) (xy 144.78 88.9)
 		)
@@
 	(wire
 		(pts
+			(xy 45.085 68.58) (xy 45.085 70.485)
+		)
+		(stroke
+			(width 0)
+			(type default)
+		)
+	)
+	(wire
+		(pts
 			(xy 170.18 48.26) (xy 170.18 68.58)
 		)
@@
 	(wire
 		(pts
-			(xy 27.94 68.58) (xy 40.64 68.58)
+			(xy 27.94 68.58) (xy 45.085 68.58)
 		)
 		(stroke
@@
 	(wire
 		(pts
+			(xy 45.085 68.58) (xy 50.165 68.58)
+		)
+		(stroke
+			(width 0)
+			(type default)
+		)
+	)
+	(wire
+		(pts
 			(xy 160.02 78.74) (xy 177.8 78.74)
 		)
@@
 	(global_label "PP4V2"
 		(shape input)
-		(at 40.64 68.58 0)
+		(at 50.165 68.58 0)
 		(fields_autoplaced yes)
 		(effects
@@
 		)
 		(property "Intersheetrefs" "${INTERSHEET_REFS}"
-			(at 49.6728 68.58 0)
+			(at 59.1978 68.58 0)
 			(hide yes)
 			(show_name no)
@@
 	)
 	(symbol
+		(lib_id "Device:C")
+		(at 45.085 74.295 180)
+		(unit 1)
+		(body_style 1)
+		(exclude_from_sim no)
+		(in_bom yes)
+		(on_board yes)
+		(in_pos_files yes)
+		(dnp no)
+		(property "Reference" "S1C1"
+			(at 59.055 80.01 0)
+			(show_name no)
+			(do_not_autoplace no)
+			(effects
+				(font
+					(size 1.27 1.27)
+				)
+			)
+		)
+		(property "Value" "0402 100nF 10V 10% X7R"
+			(at 59.055 77.47 0)
+			(show_name no)
+			(do_not_autoplace no)
+			(effects
+				(font
+					(size 1.27 1.27)
+				)
+			)
+		)
+		(property "Footprint" "Capacitor_SMD:C_0402_1005Metric"
+			(at 44.1198 70.485 0)
+			(hide yes)
+			(show_name no)
+			(do_not_autoplace no)
+			(effects
+				(font
+					(size 1.27 1.27)
+				)
+			)
+		)
+		(property "Datasheet" ""
+			(at 45.085 74.295 0)
+			(hide yes)
+			(show_name no)
+			(do_not_autoplace no)
+			(effects
+				(font
+					(size 1.27 1.27)
+				)
+			)
+		)
+		(property "Description" "Unpolarized capacitor"
+			(at 45.085 74.295 0)
+			(hide yes)
+			(show_name no)
+			(do_not_autoplace no)
+			(effects
+				(font
+					(size 1.27 1.27)
+				)
+			)
+		)
+		(pin "1"
+		)
+		(pin "2"
+		)
+		(instances
+			(project "l0destar"
+				(path "/463fa308-d92b-480b-9c45-50693d427ea2"
+					(reference "S1C1")
+					(unit 1)
+				)
+			)
+		)
+	)
+	(symbol
 		(lib_id "power:GND")
 		(at 40.64 38.1 0)
@@
 					(unit 1)
 				)
+			)
+		)
+	)
+	(symbol
+		(lib_id "power:GND")
+		(at 45.085 81.28 0)
+		(unit 1)
+		(body_style 1)
+		(exclude_from_sim no)
+		(in_bom yes)
+		(on_board yes)
+		(in_pos_files yes)
+		(dnp no)
+		(property "Reference" "#PWR060"
+			(at 45.085 87.63 0)
+			(hide yes)
+			(show_name no)
+			(do_not_autoplace no)
+			(effects
+				(font
+					(size 1.27 1.27)
+				)
+			)
+		)
+		(property "Value" "GND"
+			(at 46.863 85.344 0)
+			(show_name no)
+			(do_not_autoplace no)
+			(effects
+				(font
+					(size 1.27 1.27)
+				)
+				(justify right)
+			)
+		)
+		(property "Footprint" ""
+			(at 45.085 81.28 0)
+			(hide yes)
+			(show_name no)
+			(do_not_autoplace no)
+			(effects
+				(font
+					(size 1.27 1.27)
+				)
+			)
+		)
+		(property "Datasheet" ""
+			(at 45.085 81.28 0)
+			(hide yes)
+			(show_name no)
+			(do_not_autoplace no)
+			(effects
+				(font
+					(size 1.27 1.27)
+				)
+			)
+		)
+		(property "Description" "Power symbol creates a global label with name \"GND\" , ground"
+			(at 45.085 81.28 0)
+			(hide yes)
+			(show_name no)
+			(do_not_autoplace no)
+			(effects
+				(font
+					(size 1.27 1.27)
+				)
+			)
+		)
+		(pin "1"
+		)
+		(instances
+			(project "l0destar"
+				(path "/463fa308-d92b-480b-9c45-50693d427ea2"
+					(reference "#PWR060")
+					(unit 1)
+				)

Commit message: update v3.1
Parts:
- added S1R5: 0402 100K 5%, Resistor_SMD:R_0402_1005Metric, symbol Device:R
Connections:
- net ACCELL_INT1: now also S1J2.16 (Pin_16); no longer S1J2.15 (Pin_15)
- net CAN_CS: now also S1J3.23 (Pin_18); no longer S1J3.26 (Pin_15)
- net CAN_SCK: now also S1J3.25 (Pin_16); no longer S1J3.24 (Pin_17)
- net CAN_SDI: now also S1J3.24 (Pin_17); no longer S1J3.23 (Pin_18)
- net CAN_SDO: now also S1J3.26 (Pin_15); no longer S1J3.25 (Pin_16)
- net GND: now also S1R5.1
- net K_ENABLE: now reaches S1J3.33 (Pin_8)
- net K_ENABLE: now also S1R5.2
- net OBD_ENABLE renamed CAN_ENABLE
- net PP12V_OBD_ST renamed PP3V3_K_ST
- net PP3V3_OBD_ST renamed PP3V3_CAN_ST
- new net PP12V_K_ST: S1J2.15 (Pin_15)

Commit message: update v3.1
Parts:
- S1C1: Manufacturer_Name (none) -> Multicomp Pro; Manufacturer_Part_Number (none) -> MC0402B104K250CT
- S1J1: Manufacturer_Name (none) -> Molex; Manufacturer_Part_Number (none) -> 43045-0600
- S1R1, S1R2: Manufacturer_Name (none) -> Multicomp Pro; Manufacturer_Part_Number (none) -> MP003476
- S1R3, S1R4, S1R5: Manufacturer_Name (none) -> Multicomp Pro; Manufacturer_Part_Number (none) -> MCPWR02FTEP1003A
Changed lines of the file:
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@@
 			)
 		)
-		(property "Datasheet" ""
+		(property "Datasheet" "https://uk.farnell.com/multicomp-pro/mcpwr02ftep1003a/res-100k-1-thick-film-0402/dp/4538624"
 			(at 175.26 97.79 0)
 			(hide yes)
@@
 					(size 1.27 1.27)
 				)
+			)
+		)
+		(property "Manufacturer_Part_Number" "MCPWR02FTEP1003A"
+			(at 175.26 97.79 0)
+			(hide yes)
+			(show_name no)
+			(do_not_autoplace no)
+			(effects
+				(font
+					(size 1.27 1.27)
+				)
+				(justify left top)
+			)
+		)
+		(property "Manufacturer_Name" "Multicomp Pro"
+			(at 175.26 97.79 0)
+			(hide yes)
+			(show_name no)
+			(do_not_autoplace no)
+			(effects
+				(font
+					(size 1.27 1.27)
+				)
+				(justify left top)
 			)
 		)
@@
 			)
 		)
-		(property "Datasheet" ""
+		(property "Datasheet" "https://uk.farnell.com/multicomp-pro/mcpwr02ftep1003a/res-100k-1-thick-film-0402/dp/4538624"
 			(at 154.94 97.79 0)
 			(hide yes)
@@
 					(size 1.27 1.27)
 				)
+			)
+		)
+		(property "Manufacturer_Part_Number" "MCPWR02FTEP1003A"
+			(at 154.94 97.79 0)
+			(hide yes)
+			(show_name no)
+			(do_not_autoplace no)
+			(effects
+				(font
+					(size 1.27 1.27)
+				)
+				(justify left top)
+			)
+		)
+		(property "Manufacturer_Name" "Multicomp Pro"
+			(at 154.94 97.79 0)
+			(hide yes)
+			(show_name no)
+			(do_not_autoplace no)
+			(effects
+				(font
+					(size 1.27 1.27)
+				)
+				(justify left top)
 			)
 		)
@@
 			)
 		)
-		(property "Datasheet" ""
+		(property "Datasheet" "https://uk.farnell.com/multicomp-pro/mp003476/res-4k7-1-0-0625w-0402-thick-film/dp/3392645"
 			(at 218.44 29.21 0)
 			(hide yes)
@@
 					(size 1.27 1.27)
 				)
+			)
+		)
+		(property "Manufacturer_Part_Number" "MP003476"
+			(at 218.44 29.21 0)
+			(hide yes)
+			(show_name no)
+			(do_not_autoplace no)
+			(effects
+				(font
+					(size 1.27 1.27)
+				)
+				(justify left top)
+			)
+		)
+		(property "Manufacturer_Name" "Multicomp Pro"
+			(at 218.44 29.21 0)
+			(hide yes)
+			(show_name no)
+			(do_not_autoplace no)
+			(effects
+				(font
+					(size 1.27 1.27)
+				)
+				(justify left top)
 			)
 		)
@@
 			)
 		)
-		(property "Datasheet" ""
+		(property "Datasheet" "https://uk.farnell.com/multicomp-pro/mc0402b104k250ct/cap-0-1-f-25v-10-x7r-0402/dp/2320759"
 			(at 45.085 74.295 0)
 			(hide yes)
@@
 					(size 1.27 1.27)
 				)
+			)
+		)
+		(property "Manufacturer_Part_Number" "MC0402B104K250CT"
+			(at 45.085 74.295 0)
+			(hide yes)
+			(show_name no)
+			(do_not_autoplace no)
+			(effects
+				(font
+					(size 1.27 1.27)
+				)
+				(justify left top)
+			)
+		)
+		(property "Manufacturer_Name" "Multicomp Pro"
+			(at 45.085 74.295 0)
+			(hide yes)
+			(show_name no)
+			(do_not_autoplace no)
+			(effects
+				(font
+					(size 1.27 1.27)
+				)
+				(justify left top)
 			)
 		)
@@
 			)
 		)
-		(property "Datasheet" ""
+		(property "Datasheet" "https://uk.farnell.com/multicomp-pro/mcpwr02ftep1003a/res-100k-1-thick-film-0402/dp/4538624"
 			(at 199.39 62.23 0)
 			(hide yes)
@@
 					(size 1.27 1.27)
 				)
+			)
+		)
+		(property "Manufacturer_Part_Number" "MCPWR02FTEP1003A"
+			(at 199.39 62.23 0)
+			(hide yes)
+			(show_name no)
+			(do_not_autoplace no)
+			(effects
+				(font
+					(size 1.27 1.27)
+				)
+				(justify left top)
+			)
+		)
+		(property "Manufacturer_Name" "Multicomp Pro"
+			(at 199.39 62.23 0)
+			(hide yes)
+			(show_name no)
+			(do_not_autoplace no)
+			(effects
+				(font
+					(size 1.27 1.27)
+				)
+				(justify left top)
 			)
 		)
@@
 			)
 		)
-		(property "Datasheet" ""
+		(property "Datasheet" "https://www.molex.com/content/dam/molex/molex-dot-com/products/automated/en-us/productspecificationpdf/430/43045/PS-43045-001.pdf"
 			(at 48.26 30.48 0)
 			(hide yes)
@@
 					(size 1.27 1.27)
 				)
+			)
+		)
+		(property "Manufacturer_Part_Number" "43045-0600"
+			(at 48.26 30.48 0)
+			(hide yes)
+			(show_name no)
+			(do_not_autoplace no)
+			(effects
+				(font
+					(size 1.27 1.27)
+				)
+				(justify left top)
+			)
+		)
+		(property "Manufacturer_Name" "Molex"
+			(at 48.26 30.48 0)
+			(hide yes)
+			(show_name no)
+			(do_not_autoplace no)
+			(effects
+				(font
+					(size 1.27 1.27)
+				)
+				(justify left top)
 			)
 		)
@@
 			)
 		)
-		(property "Datasheet" ""
+		(property "Datasheet" "https://uk.farnell.com/multicomp-pro/mp003476/res-4k7-1-0-0625w-0402-thick-film/dp/3392645"
 			(at 198.12 29.21 0)
 			(hide yes)
@@
 			)
 		)
+		(property "Manufacturer_Part_Number" "MP003476"
+			(at 198.12 29.21 0)
+			(hide yes)
+			(show_name no)
+			(do_not_autoplace no)
+			(effects
+				(font
+					(size 1.27 1.27)
+				)
+				(justify left top)
+			)
+		)
+		(property "Manufacturer_Name" "Multicomp Pro"
+			(at 198.12 29.21 0)
+			(hide yes)
+			(show_name no)
+			(do_not_autoplace no)
+			(effects
+				(font
+					(size 1.27 1.27)
+				)
+				(justify left top)
+			)
+		)

Commit message: update sheet annotations
Other:
- note added: "19/08/2026"
- note added: "3.1"
- note added: "Main external connector 6-pin Microfit 3.0 40-pin dual header for the MakerDiary nRF9151 Connect Kit Makerdiary power cable connection point with 100nF decoupling I2C pullups Power rail enable pin pulldowns"
- note removed: "1.0"
- note removed: "30/05/2026"
- note removed: "Main connector 40-pin dual header for the MakerDiary nRF9151 Connect Kit Makerdiary power cable connection point with ceramic bulk Jumper pads for CAN / ISO-9141 configuration"
Changed lines of the file:
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@@
 		)
 	)
-	(text "Main connector\n40-pin dual header for the MakerDiary nRF9151 Connect Kit\nMakerdiary power cable connection point with ceramic bulk\nJumper pads for CAN / ISO-9141 configuration"
+	(text "Main external connector 6-pin Microfit 3.0\n40-pin dual header for the MakerDiary nRF9151 Connect Kit\nMakerdiary power cable connection point with 100nF decoupling\nI2C pullups\nPower rail enable pin pulldowns"
 		(exclude_from_sim no)
-		(at 180.848 173.228 0)
+		(at 179.705 172.72 0)
 		(effects
 			(font
@@
 		)
 	)
-	(text "30/05/2026"
+	(text "19/08/2026"
 		(exclude_from_sim no)
 		(at 205.994 193.294 0)
@@
 		)
 	)
-	(text "1.0"
+	(text "3.1"
 		(exclude_from_sim no)
 		(at 268.478 193.294 0)

Commit message: schematic<>readme discrepency fixes
Parts:
- S1C1: value 0402 100nF 10V 10% X7R -> 0402 100nF 50V 10% X7R; Manufacturer_Name Multicomp Pro -> Murata; Manufacturer_Part_Number MC0402B104K250CT -> GRM155R71H104KE14D
Changed lines of the file:
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@@
 			)
 		)
-		(property "Value" "0402 100nF 10V 10% X7R"
+		(property "Value" "0402 100nF 50V 10% X7R"
 			(at 59.055 77.47 0)
 			(show_name no)
@@
 			)
 		)
-		(property "Datasheet" "https://uk.farnell.com/multicomp-pro/mc0402b104k250ct/cap-0-1-f-25v-10-x7r-0402/dp/2320759"
+		(property "Datasheet" ""
 			(at 45.085 74.295 0)
 			(hide yes)
@@
 			)
 		)
-		(property "Manufacturer_Part_Number" "MC0402B104K250CT"
+		(property "Manufacturer_Part_Number" "GRM155R71H104KE14D"
 			(at 45.085 74.295 0)
 			(hide yes)
@@
 			)
 		)
-		(property "Manufacturer_Name" "Multicomp Pro"
+		(property "Manufacturer_Name" "Murata"
 			(at 45.085 74.295 0)
 			(hide yes)
