File: hardware/l0destar_v3.3/can_interface.kicad_sch (KiCad schematic)
At the start: 18 parts

Commit message: schematic<>readme discrepency fixes
Parts:
- S9C1, S9C4: value 0402 100nF 10V 10% X7R -> 0402 100nF 50V 10% X7R; Manufacturer_Name Multicomp Pro -> Murata; Manufacturer_Part_Number MC0402B104K250CT -> GRM155R71H104KE14D
Changed lines of the file:
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@@
 			)
 		)
-		(property "Value" "0402 100nF 10V 10% X7R"
+		(property "Value" "0402 100nF 50V 10% X7R"
 			(at 150.114 120.904 0)
 			(show_name no)
@@
 			)
 		)
-		(property "Datasheet" "https://uk.farnell.com/multicomp-pro/mc0402b104k250ct/cap-0-1-f-25v-10-x7r-0402/dp/2320759"
+		(property "Datasheet" ""
 			(at 147.32 119.38 0)
 			(hide yes)
@@
 			)
 		)
-		(property "Description" "Unpolarized capacitor"
+		(property "Description" ""
 			(at 147.32 119.38 0)
 			(hide yes)
@@
 			)
 		)
-		(property "Manufacturer_Part_Number" "MC0402B104K250CT"
+		(property "Manufacturer_Part_Number" "GRM155R71H104KE14D"
 			(at 147.32 119.38 0)
 			(hide yes)
@@
 			)
 		)
-		(property "Manufacturer_Name" "Multicomp Pro"
+		(property "Manufacturer_Name" "Murata"
 			(at 147.32 119.38 0)
 			(hide yes)
@@
 			)
 		)
-		(property "Value" "0402 100nF 10V 10% X7R"
+		(property "Value" "0402 100nF 50V 10% X7R"
 			(at 48.26 71.755 0)
 			(show_name no)
@@
 			)
 		)
-		(property "Datasheet" "https://uk.farnell.com/multicomp-pro/mc0402b104k250ct/cap-0-1-f-25v-10-x7r-0402/dp/2320759"
+		(property "Datasheet" ""
 			(at 68.58 55.88 0)
 			(hide yes)
@@
 			)
 		)
-		(property "Description" "Unpolarized capacitor"
+		(property "Description" ""
 			(at 68.58 55.88 0)
 			(hide yes)
@@
 			)
 		)
-		(property "Manufacturer_Part_Number" "MC0402B104K250CT"
+		(property "Manufacturer_Part_Number" "GRM155R71H104KE14D"
 			(at 68.58 55.88 0)
 			(hide yes)
@@
 			)
 		)
-		(property "Manufacturer_Name" "Multicomp Pro"
+		(property "Manufacturer_Name" "Murata"
 			(at 68.58 55.88 0)
 			(hide yes)
