File: hardware/l0destar_v3.3/battery_voltage_reading.kicad_sch (KiCad schematic)
At the start: 3 parts

Commit message: schematic<>readme discrepency fixes
Parts:
- S3C1: value 0402 1uF 10V 10% X7R -> 0603 2.2uF 25V 10% X7R; footprint Capacitor_SMD:C_0402_1005Metric -> Resistor_SMD:R_0603_1608Metric
- S3C2: value 0402 100nF 10V 10% X7R -> 0402 100nF 50V 10% X7R; Manufacturer_Name Multicomp Pro -> Murata; Manufacturer_Part_Number MC0402B104K250CT -> GRM155R71H104KE14D
Other:
- note added: "Vehicle voltage reading via INA228 using the I2C bus 100nF / 2.2uF decoupling"
- note removed: "Vehicle voltage reading via INA228 using the I2C bus 100nF / 1uF decoupling"
Changed lines of the file:
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@@
 		)
 	)
-	(text "Vehicle voltage reading via INA228 using the I2C bus\n100nF / 1uF decoupling"
+	(text "Vehicle voltage reading via INA228 using the I2C bus\n100nF / 2.2uF decoupling"
 		(exclude_from_sim no)
 		(at 179.07 169.545 0)
@@
 			)
 		)
-		(property "Value" "0402 1uF 10V 10% X7R"
+		(property "Value" "0603 2.2uF 25V 10% X7R"
 			(at 112.395 48.895 0)
 			(show_name no)
@@
 			)
 		)
-		(property "Footprint" "Capacitor_SMD:C_0402_1005Metric"
+		(property "Footprint" "Resistor_SMD:R_0603_1608Metric"
 			(at 114.6048 57.15 0)
 			(hide yes)
@@
 			)
 		)
-		(property "Value" "0402 100nF 10V 10% X7R"
+		(property "Value" "0402 100nF 50V 10% X7R"
 			(at 147.32 48.895 0)
 			(show_name no)
@@
 			)
 		)
-		(property "Datasheet" "https://uk.farnell.com/multicomp-pro/mc0402b104k250ct/cap-0-1-f-25v-10-x7r-0402/dp/2320759"
+		(property "Datasheet" ""
 			(at 144.145 60.96 0)
 			(hide yes)
@@
 			)
 		)
-		(property "Description" "Unpolarized capacitor"
+		(property "Description" ""
 			(at 144.145 60.96 0)
 			(hide yes)
@@
 			)
 		)
-		(property "Manufacturer_Part_Number" "MC0402B104K250CT"
+		(property "Manufacturer_Part_Number" "GRM155R71H104KE14D"
 			(at 144.145 60.96 0)
 			(hide yes)
@@
 			)
 		)
-		(property "Manufacturer_Name" "Multicomp Pro"
+		(property "Manufacturer_Name" "Murata"
 			(at 144.145 60.96 0)
 			(hide yes)

Commit message: revised 3.3 board, parts and readme updates
Parts:
- S3C1: footprint Resistor_SMD:R_0603_1608Metric -> Capacitor_SMD:C_0603_1608Metric
Changed lines of the file:
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@@
 			)
 		)
-		(property "Footprint" "Resistor_SMD:R_0603_1608Metric"
+		(property "Footprint" "Capacitor_SMD:C_0603_1608Metric"
 			(at 114.6048 57.15 0)
 			(hide yes)
