File: hardware/l0destar_v3.3/auxillary_power_control.kicad_sch (KiCad schematic)
At the start: 23 parts

Commit message: schematic<>readme discrepency fixes
Parts:
- S7C1, S7C3, S7C8: value 0402 1uF 10V 10% X7R -> 0603 2.2uF 25V 10% X7R; footprint Capacitor_SMD:C_0402_1005Metric -> Resistor_SMD:R_0603_1608Metric
- S7C2, S7C4, S7C9: value 0402 100nF 10V 10% X7R -> 0402 100nF 50V 10% X7R; Manufacturer_Name Multicomp Pro -> Murata; Manufacturer_Part_Number MC0402B104K250CT -> GRM155R71H104KE14D
Other:
- moved on the sheet: S7C8, S7C9, S7R8, S7R9, S7U4

Commit message: revised 3.3 board, parts and readme updates
Parts:
- S7C1, S7C3, S7C8: footprint Resistor_SMD:R_0603_1608Metric -> Capacitor_SMD:C_0603_1608Metric
Changed lines of the file:
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@@
 			)
 		)
-		(property "Footprint" "Resistor_SMD:R_0603_1608Metric"
+		(property "Footprint" "Capacitor_SMD:C_0603_1608Metric"
 			(at 35.2552 111.125 0)
 			(hide yes)
@@
 			)
 		)
-		(property "Footprint" "Resistor_SMD:R_0603_1608Metric"
+		(property "Footprint" "Capacitor_SMD:C_0603_1608Metric"
 			(at 35.2552 38.735 0)
 			(hide yes)
@@
 			)
 		)
-		(property "Footprint" "Resistor_SMD:R_0603_1608Metric"
+		(property "Footprint" "Capacitor_SMD:C_0603_1608Metric"
 			(at 35.2552 74.295 0)
 			(hide yes)

Commit message: change resistor divider and a few parts
Other:
- note added: "Load switches for auxilliary power rails GPS / 3.3V CAN / 3.3V K / 12V K (typically only one of CAN/K will be present) State signals via GPIO for rail fault detection 12V state signal is inverted by its MOSFET"
- note added: "l0destar auxilliary power control"
- note removed: "Load switches for auxillary power rails GPS / 3.3V CAN / 3.3V K / 12V K (typically only one of CAN/K will be present) State signals via GPIO for rail fault detection 12V state signal is inverted by its MOSFET"
- note removed: "l0destar auxillary power control"
Changed lines of the file:
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@@
 		)
 	)
-	(text "l0destar auxillary power control"
+	(text "l0destar auxilliary power control"
 		(exclude_from_sim no)
 		(at 185.928 189.738 0)
@@
 		)
 	)
-	(text "Load switches for auxillary power rails\nGPS / 3.3V CAN / 3.3V K / 12V K (typically only one of CAN/K will be present)\nState signals via GPIO for rail fault detection\n12V state signal is inverted by its MOSFET"
+	(text "Load switches for auxilliary power rails\nGPS / 3.3V CAN / 3.3V K / 12V K (typically only one of CAN/K will be present)\nState signals via GPIO for rail fault detection\n12V state signal is inverted by its MOSFET"
 		(exclude_from_sim no)
 		(at 179.705 172.72 0)
