File: hardware/l0destar_v3.3/accelerometer.kicad_sch (KiCad schematic)
At the start: 7 parts

Commit message: schematic<>readme discrepency fixes
Parts:
- S8C1, S8C3: value 0402 100nF 10V 10% X7R -> 0402 100nF 50V 10% X7R; Manufacturer_Name Multicomp Pro -> Murata; Manufacturer_Part_Number MC0402B104K250CT -> GRM155R71H104KE14D
- S8R1: renamed from S7R10; value 0402 0R / FB BLM15AG601SH1D -> 0402 FB BLM15AG601SH1D; Manufacturer_Name Panasonic -> (none); Manufacturer_Part_Number ERJ2RKF1004X -> BLM15AG601SH1D
Other:
- moved on the sheet: S8C1, S8C2, S8C3, S8C4, S8C5, S8R1, S8U1

Commit message: revised 3.3 board, parts and readme updates
Parts:
- S8R1: value 0402 FB BLM15AG601SH1D -> 0402 FB BLM15AG601SN1D; Manufacturer_Name (none) -> Murata; Manufacturer_Part_Number BLM15AG601SH1D -> BLM15AG601SN1D
Changed lines of the file:
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@@
 			)
 		)
-		(property "Value" "0402 FB BLM15AG601SH1D"
+		(property "Value" "0402 FB BLM15AG601SN1D"
 			(at 182.88 27.305 90)
 			(show_name no)
@@
 			)
 		)
-		(property "Datasheet" "https://industrial.panasonic.com/cdbs/www-data/pdf/RDA0000/AOA0000C304.pdf"
+		(property "Datasheet" ""
 			(at 182.88 30.48 0)
 			(hide yes)
@@
 			)
 		)
-		(property "Manufacturer_Part_Number" "BLM15AG601SH1D"
+		(property "Manufacturer_Part_Number" "BLM15AG601SN1D"
 			(at 182.88 30.48 0)
 			(hide yes)
@@
 			)
 		)
-		(property "Manufacturer_Name" ""
+		(property "Manufacturer_Name" "Murata"
 			(at 182.88 30.48 0)
 			(hide yes)

Commit message: update with new ferrite bead part number
Parts:
- S8R1: value 0402 FB BLM15AG601SN1D -> 0402 FB BLM15AG601SH1D; Manufacturer_Part_Number BLM15AG601SN1D -> BLM15AG601SH1D
Changed lines of the file:
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@@
 			)
 		)
-		(property "Value" "0402 FB BLM15AG601SN1D"
+		(property "Value" "0402 FB BLM15AG601SH1D"
 			(at 182.88 27.305 90)
 			(show_name no)
@@
 			)
 		)
-		(property "Manufacturer_Part_Number" "BLM15AG601SN1D"
+		(property "Manufacturer_Part_Number" "BLM15AG601SH1D"
 			(at 182.88 30.48 0)
 			(hide yes)

Commit message: v3.3 RF optimisation
Other:
- note removed: "0R jumper or ferrite bead if peak TX causes reading offsets"
Changed lines of the file:
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@@
-		)
-	)
-	(text "0R jumper or ferrite bead if peak TX causes reading offsets"
-		(exclude_from_sim no)
-		(at 182.88 19.685 0)
-		(effects
-			(font
-				(size 1.27 1.27)
-			)
 		)
 	)
