File: hardware/l0destar_v3.3/test_points.kicad_sch (KiCad schematic)
At the start: 9 parts

Commit message: v3.3 minor layout tweaks
Parts:
- removed S12TP1: 3.3V, TestPoint:TestPoint_Pad_1.0x1.0mm, symbol Connector:TestPoint
- removed S12TP2: 3.3V GPS, TestPoint:TestPoint_Pad_1.0x1.0mm, symbol Connector:TestPoint
- removed S12TP3: 12V protected, TestPoint:TestPoint_Pad_1.0x1.0mm, symbol Connector:TestPoint
- removed S12TP4: 3.3V CAN, TestPoint:TestPoint_Pad_1.0x1.0mm, symbol Connector:TestPoint
- removed S12TP5: 3.3V K, TestPoint:TestPoint_Pad_1.0x1.0mm, symbol Connector:TestPoint
