File: hardware/l0destar_v3.4/kwire_interface.kicad_sch (KiCad schematic)
At the start: 18 parts

Commit message: change references to ISO-9141 to k-wire
Other:
- note added: "K-wire interface using TJA1027T TVS on the K and L wires L line can be pulled low via L_SEND AL5809-90 added to limit current to 90mA in the event that L is shorted to 12V Sense signal added to detect short to 12V on the L line"
- note added: "l0destar k-wire interface"
- note removed: "ISO-9141 interface (K-line) using TJA1027T TVS on the K and L wires L line can be pulled low via L_SEND AL5809-90 added to limit current to 90mA in the event that L is shorted to 12V Sense signal added to detect short to 12V on the L line"
- note removed: "l0destar ISO-9141 interface"
Changed lines of the file:
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@@
 	(generator_version "10.0")
 	(paper "A4")
-	(text "l0destar ISO-9141 interface"
+	(text "l0destar k-wire interface"
 		(exclude_from_sim no)
 		(at 186.436 189.738 0)
@@
 		)
 	)
-	(text "ISO-9141 interface (K-line) using TJA1027T\nTVS on the K and L wires\nL line can be pulled low via L_SEND\nAL5809-90 added to limit current to 90mA in the event that L is shorted to 12V\nSense signal added to detect short to 12V on the L line"
+	(text "K-wire interface using TJA1027T\nTVS on the K and L wires\nL line can be pulled low via L_SEND\nAL5809-90 added to limit current to 90mA in the event that L is shorted to 12V\nSense signal added to detect short to 12V on the L line"
 		(exclude_from_sim no)
 		(at 179.07 173.355 0)
