File: hardware/l0destar_v3.4/l0destar.kicad_sch (KiCad schematic)
At the start: 10 parts

Commit message: update v3.4
Parts:
- S1J4: footprint libs:Makerdiary_power_header -> libs:MakerDiary2PinHeader
Changed lines of the file:
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@@
 			)
 		)
-		(property "Footprint" "libs:Makerdiary_power_header"
+		(property "Footprint" "libs:MakerDiary2PinHeader"
 			(at 22.86 68.58 0)
 			(hide yes)

Commit message: change references to ISO-9141 to k-wire
Connections:
- net CAN_H_ISO9141_K renamed CAN_H_KWIRE_K
- net CAN_L_ISO9141_L renamed CAN_L_KWIRE_L
Changed lines of the file:
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@@
 		)
 	)
-	(global_label "CAN_H_ISO9141_K"
+	(global_label "CAN_H_KWIRE_K"
 		(shape input)
 		(at 38.1 33.02 180)
@@
 		)
 		(property "Intersheetrefs" "${INTERSHEET_REFS}"
-			(at 17.9396 33.02 0)
+			(at 20.1772 33.02 0)
 			(hide yes)
 			(show_name no)
@@
 		)
 	)
-	(global_label "CAN_L_ISO9141_L"
+	(global_label "CAN_L_KWIRE_L"
 		(shape input)
 		(at 60.96 27.94 0)
@@
 		)
 		(property "Intersheetrefs" "${INTERSHEET_REFS}"
-			(at 80.5761 27.94 0)
-			(hide yes)
-			(show_name no)
+			(at 78.3385 27.94 0)
+			(hide yes)
+			(show_name no)
