File: hardware/l0destar_v3.4/can_interface.kicad_sch (KiCad schematic)
At the start: 18 parts

Commit message: cleanup and chip swap
Parts:
- S9U1: value MAX33041EASA+ -> TCAN3414DR; footprint libs:SOIC127P600X175-8N -> SOIC127P600X175-8N; symbol MAX33041EASA+:MAX33041EASA+ -> TCAN3414DR:TCAN3414DR; Manufacturer_Part_Number MAX33041EASA+ -> TCAN3414DR
Changed lines of the file:
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@@
 	)
 	(symbol
-		(lib_id "MAX33041EASA+:MAX33041EASA+")
+		(lib_id "TCAN3414DR:TCAN3414DR")
 		(at 81.28 41.91 0)
 		(unit 1)
@@
 			)
 		)
-		(property "Value" "MAX33041EASA+"
+		(property "Value" "TCAN3414DR"
 			(at 95.25 36.83 0)
 			(show_name no)
@@
 			)
 		)
-		(property "Footprint" "libs:SOIC127P600X175-8N"
+		(property "Footprint" "SOIC127P600X175-8N"
 			(at 105.41 136.83 0)
 			(hide yes)
@@
 			)
 		)
-		(property "Manufacturer_Part_Number" "MAX33041EASA+"
+		(property "Manufacturer_Part_Number" "TCAN3414DR"
 			(at 105.41 836.83 0)
 			(hide yes)
