File: hardware/l0destar_v3.4/can_interface.kicad_sch (KiCad schematic)
At the start: 18 parts

Commit message: hardware: v3.4's S9U1 is fitted, with the TCAN3414's details
The board marked S9U1 as do-not-populate while the schematic did not, so a
BOM or placement file made from the board with DNP parts excluded left the CAN
transceiver off. Its datasheet link and description were still the Maxim
MAX33040E/41E's, in the schematic, its embedded symbol and
libs/TCAN3414DR.kicad_sym, and the schematic's footprint field lacked the libs:
library the board uses.

Checked with kicad-cli 10: the placement file with DNP parts excluded now
lists S9U1, and the schematic BOM carries TI's datasheet and description.

Co-Authored-By: Claude Opus 5 (1M context) <noreply@anthropic.com>
Claude-Session: https://claude.ai/code/session_018qedd7M9dswRwiNYyPeaoJ
Parts:
- S9U1: footprint SOIC127P600X175-8N -> libs:SOIC127P600X175-8N
Changed lines of the file:
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@@
 			)
 		)
-		(property "Footprint" "SOIC127P600X175-8N"
+		(property "Footprint" "libs:SOIC127P600X175-8N"
 			(at 105.41 136.83 0)
 			(hide yes)
@@
 			)
 		)
-		(property "Datasheet" "https://datasheets.maximintegrated.com/en/ds/MAX33040E-MAX33041E.pdf"
+		(property "Datasheet" "https://www.ti.com/lit/ds/symlink/tcan3414.pdf"
 			(at 105.41 236.83 0)
 			(hide yes)
@@
 			)
 		)
-		(property "Description" "+3.3V, 5Mbps CAN Transceiver with ?40V Fault Protection"
+		(property "Description" "3.3-V CAN FD transceiver with shut-down and standby mode"
 			(at 81.28 41.91 0)
 			(hide yes)
