File: hardware/l0destar_v3.4/l0destar.kicad_pcb (KiCad board)
At the start: 4 copper layers, 66.7 x 37.5 mm, 156 parts

Commit message: update v3.4
Parts:
- removed S11TP1: TestPoint - fault injection, TestPoint:TestPoint_Pad_1.0x1.0mm
- added S12TP1: GND, TestPoint:TestPoint_Pad_1.0x1.0mm, F.Cu at (25.4, 91.6)
- added S12TP3: 3.3V, TestPoint:TestPoint_Pad_1.0x1.0mm, F.Cu at (75.3, 73.1)
- added S12TP4: 3.3V GPS, TestPoint:TestPoint_Pad_1.0x1.0mm, F.Cu at (77.5, 73.1)
- added S12TP5: 3.3V CAN, TestPoint:TestPoint_Pad_1.0x1.0mm, F.Cu at (79.7, 73.1)
- added S12TP6: 3.3V K, TestPoint:TestPoint_Pad_1.0x1.0mm, F.Cu at (81.8, 87.8)
- S12TP7: value 4.2V unprotected -> 12V K
- S1J4: footprint libs:Makerdiary_power_header -> libs:MakerDiary2PinHeader
- moved S12TP7 45.7 mm to (83.9, 87.8)
- moved S1J4 0.95 mm to (26.0, 98.2)
- renumbered S12TP6 to S12TP2
Connections:
- S12TP7 pad 1: PP4V2_UNPROTECTED -> PP12V_K
Routing:
- net PP3V3_K: track 15.6 -> 43.8 mm, vias 2 -> 4
- net PP3V3: track 111.0 -> 133.7 mm
- net PP3V3_CAN: track 35.0 -> 49.1 mm
- net PP3V3_GPS: track 6.31 -> 15.5 mm
- net PP12V_K: track 40.4 -> 47.4 mm
- net PP4V2_UNPROTECTED: track 51.7 -> 46.9 mm
- net PP12VIP: track 14.3 -> 16.6 mm
- net GND: track 140.6 -> 142.4 mm, vias 194 -> 196
- net Net-(S11D1-A): track 16.0 -> 14.3 mm
- net PP4V2: track 17.8 -> 17.1 mm
Other:
- board text added: "+"
- board text added: "-"

Commit message: change references to ISO-9141 to k-wire
Connections:
- net CAN_H_ISO9141_K renamed CAN_H_KWIRE_K
- net CAN_L_ISO9141_L renamed CAN_L_KWIRE_L

Commit message: DNP the enable divider by default
Parts:
- S6R4: value 0402 1M 1% ANTI-SULFUR AEC-Q200 -> 0402 0R JUMPER OR 1M 1% ANTI-SULFUR AEC-Q200
- S6R5: value 0402 243K 1% ANTI-SULFUR AEC-Q200 -> DNP 0402 243K 1% ANTI-SULFUR AEC-Q200
- S6R6: value 0402 3.92M 1% -> DNP 0402 3.92M 1%

Commit message: cleanup and chip swap
Parts:
- S9U1: value MAX33041EASA+ -> TCAN3414DR
