File: hardware/l0destar_v3.4/antenna_bias_tee.kicad_sch (KiCad schematic)
At the start: 13 parts

Commit message: swap INA228 for INA238
Parts:
- S15D1, S15D2: value TPD1E05U06DPYR -> DNP - TPD1E05U06DPYR; now not fitted
Changed lines of the file:
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@@
 		(on_board yes)
 		(in_pos_files yes)
-		(dnp no)
+		(dnp yes)
 		(fields_autoplaced yes)
 		(property "Reference" "S15D1"
@@
 			)
 		)
-		(property "Value" "TPD1E05U06DPYR"
+		(property "Value" "DNP - TPD1E05U06DPYR"
 			(at 86.36 33.655 0)
 			(show_name no)
@@
 		(on_board yes)
 		(in_pos_files yes)
-		(dnp no)
+		(dnp yes)
 		(fields_autoplaced yes)
 		(property "Reference" "S15D2"
@@
 			)
 		)
-		(property "Value" "TPD1E05U06DPYR"
+		(property "Value" "DNP - TPD1E05U06DPYR"
 			(at 118.11 109.22 0)
 			(show_name no)
